File: led-processor-board.kicad_pcb (KiCad board)
At the start: 2 copper layers, 100 x 89.5 mm, 127 parts, among them J1 USB-C, J2 SPARE, J3 SWD, J4 12V IN, J5 OUT1, J6 OUT2, J7 OUT3, J8 OUT4, J9 WL_GPIO, SW1 TS-1088R-02526, SW2 TS-1088R-02526, U1 RP2350B, U2 NCP1117ST33T3G, U3 W25Q128JVSIQ, U4 APS6404L-3SQR-SN, U5 RM2, U6 DS3231SN, U7 TPS54202H, X1 12MHz

Commit message: Added labels to the UART RX and TX that we'll need to use for debugging
Routing:
- net /GPIO0: track 41.5 -> 37.2 mm
- net /GPIO1: track 38.3 -> 35.7 mm
Other:
- board text added: "U1 RX"
- board text added: "U1 TX"
