File: led-processor-board.kicad_pcb (KiCad board)
At the start: 2 copper layers, 100 x 89.5 mm, 127 parts, among them J1 USB-C, J2 SPARE, J3 SWD, J4 12V IN, J5 OUT1, J6 OUT2, J7 OUT3, J8 OUT4, J9 WL_GPIO, SW1 TS-1088R-02526, SW2 TS-1088R-02526, U1 RP2350B, U2 NCP1117ST33T3G, U3 W25Q128JVSIQ, U4 APS6404L-3SQR-SN, U5 RM2, U6 DS3231SN, U7 TPS54202H, X1 12MHz

Commit message: Add the SJG big-brother logo to the silkscreen
The chip guy holding hands with two LED guys (the output board's mascot),
16 mm tall, in the empty space left of the RP2350 at (79, 113). Source SVG
in docs/logo/; tools/pcb/svg_logo.py turns it into logos.pretty/
SJG_BigBrother.kicad_mod (filled F.SilkS polygons, board-only, excluded
from BOM and position files). DRC: no new items.

Co-Authored-By: Claude Opus 5.5 <noreply@anthropic.com>
Claude-Session: https://claude.ai/code/session_01NSi48cydvQ6UvBo4im78hn
Parts:
- added G1: SJG_BigBrother, logos:SJG_BigBrother, F.Cu at (79.0, 113.0)
