File: Power.kicad_sch (KiCad schematic)
At the start: 18 parts, among them J4 12V IN, U7 TPS54202H

Commit message: Use a USB-C receptacle instead of the micro-B
J1 is now a Korean Hroparts TYPE-C-31-M-12 (LCSC C165948, stock KiCad
footprint), USB 2.0: D+/D- from both sides joined, 5.1k pull-downs on
CC1/CC2 (R56, R57), SBU unconnected, shell to GND. VBUS still feeds D2.
PWR_FLAGs on VBUS and GND replace the drive the old symbol's power pins
gave; ERC is unchanged (only Pi's inherited items).

Co-Authored-By: Claude Opus 5.5 (1M context) <noreply@anthropic.com>
Claude-Session: https://claude.ai/code/session_01CYnkeL97vxsPSCyXSKGro9
Parts:
- removed C28: 10u, Capacitor_SMD:C_0805_2012Metric, symbol Device:C
- removed D3: SS34, Diode_SMD:D_SMA, symbol Device:D_Schottky
- removed R20: 510k, Resistor_SMD:R_0402_1005Metric, symbol Device:R
- added C33: 22u, Capacitor_SMD:C_0805_2012Metric, symbol Device:C
- added L2: 15u, Inductor_SMD:L_Sunlord_SWPA8040S, symbol Device:L
- added R22: 13.3k, Resistor_SMD:R_0402_1005Metric, symbol Device:R
- C28: renamed from R22; value 13.3k -> 10u; footprint Resistor_SMD:R_0402_1005Metric -> Capacitor_SMD:C_0805_2012Metric; symbol Device:R -> Device:C; LCSC C122547 -> C440198; manufacturer UNI-ROYAL -> Samsung; manufacturer_pn 0402WGF1332TCE -> CL21A106KBYNNNE
- D3: renamed from L2; value 15u -> SS34; footprint Inductor_SMD:L_Sunlord_SWPA8040S -> Diode_SMD:D_SMA; symbol Device:L -> Device:D_Schottky; LCSC C16853 -> C8678; manufacturer Sunlord -> MDD; manufacturer_pn SWPA8040S150MT -> SS34
- R20: renamed from C33; value 22u -> 510k; footprint Capacitor_SMD:C_0805_2012Metric -> Resistor_SMD:R_0402_1005Metric; symbol Device:C -> Device:R; LCSC C45783 -> C11616; manufacturer Samsung -> UNI-ROYAL; manufacturer_pn CL21A226MAQNNNE -> 0402WGF5103TCE
Connections:
- net +12V: now also C28.1, D3.1 (K), R20.1
- net +5V: now also C33.1, L2.2; no longer D3.2, R20.1
- net FB: now also R22.1; no longer C28.1
- net GND: now also C33.2, R22.2; no longer R20.2
- net SW: now also L2.1; no longer D3.1
- net VIN_RAW: now also D3.2 (A)
- net at U7.5 (EN): now also R20.2

Commit message: Swap D1/D5 to KENTO KT-0603YG (C2289)
The Everlight green LED (C72043) is short at JLC. KT-0603YG is a
yellow-green 0603 with a 2.0-2.2 V forward drop, so D1 (WL_GPIO0, 3.3 V)
and D5 (+5V) through their 1k resistors are brighter than before.
Schematic, board fields and bom-full.csv updated; DRC parity clean.

Co-Authored-By: Claude Opus 5.5 (1M context) <noreply@anthropic.com>
Claude-Session: https://claude.ai/code/session_01CYnkeL97vxsPSCyXSKGro9
Parts:
- D5: LCSC C72043 -> C2289; manufacturer Everlight -> Hubei KENTO Elec; manufacturer_pn 19-217/GHC-YR1S2/3T -> KT-0603YG
Changed lines of the file:
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@@
 			)
 		)
-		(property "manufacturer" "Everlight"
+		(property "manufacturer" "Hubei KENTO Elec"
 			(at 193.04 97.79 0)
 			(hide yes)
@@
 			)
 		)
-		(property "manufacturer_pn" "19-217/GHC-YR1S2/3T"
+		(property "manufacturer_pn" "KT-0603YG"
 			(at 193.04 97.79 0)
 			(hide yes)
@@
 			)
 		)
-		(property "LCSC" "C72043"
+		(property "LCSC" "C2289"
 			(at 193.04 97.79 0)
 			(hide yes)
