File: led-processor-board.kicad_sch (KiCad schematic)
At the start: 68 parts, among them J1 USB-C, J2 SPARE, J3 SWD, J9 WL_GPIO, SW1 TS-1088R-02526, SW2 TS-1088R-02526, U1 RP2350B, U2 NCP1117ST33T3G, U3 W25Q128JVSIQ, U4 APS6404L-3SQR-SN, U5 RM2, U6 DS3231SN, X1 12MHz

Commit message: Swap D1/D5 to KENTO KT-0603YG (C2289)
The Everlight green LED (C72043) is short at JLC. KT-0603YG is a
yellow-green 0603 with a 2.0-2.2 V forward drop, so D1 (WL_GPIO0, 3.3 V)
and D5 (+5V) through their 1k resistors are brighter than before.
Schematic, board fields and bom-full.csv updated; DRC parity clean.

Co-Authored-By: Claude Opus 5.5 (1M context) <noreply@anthropic.com>
Claude-Session: https://claude.ai/code/session_01CYnkeL97vxsPSCyXSKGro9
Parts:
- D1: LCSC C72043 -> C2289; manufacturer Everlight -> Hubei KENTO Elec; manufacturer_pn 19-217/GHC-YR1S2/3T -> KT-0603YG
Changed lines of the file:
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@@
 			)
 		)
-		(property "manufacturer" "Everlight"
+		(property "manufacturer" "Hubei KENTO Elec"
 			(at 80.01 92.71 0)
 			(hide yes)
@@
 			)
 		)
-		(property "manufacturer_pn" "19-217/GHC-YR1S2/3T"
+		(property "manufacturer_pn" "KT-0603YG"
 			(at 80.01 92.71 0)
 			(hide yes)
@@
 			)
 		)
-		(property "LCSC" "C72043"
+		(property "LCSC" "C2289"
 			(at 80.01 92.71 0)
 			(hide yes)
